Commit message: Add files via upload

File: x1_description/urdf/mercury_x1.urdf (robot description, URDF)
Before this commit: robot firefighter, 19 links, 18 joints
Joints:
- joint joint6_L: limit lower=-1.9198 upper=3.0543 effort=1000.0 velocity=2.0 -> lower=-1.9198 upper=3.0543 effort=1000.0 velocity=0.0
- joint joint6_R: limit lower=-1.9198 upper=3.0543 effort=1000.0 velocity=2.0 -> lower=-1.9198 upper=3.0543 effort=1000.0 velocity=0.0
